File: PCB/main.brd (EAGLE design)
At the start: 76.2 x 50.8 mm, 19 parts

Commit message: Updated PCB
Parts:
- removed SDCARD1: ADAFRUIT_SDCARD3V3THROUGHHOLE, TeelSys-0.3:ADAFRUIT_SDCARD3V3
- added C2: 0.1 uF, microbuilder:_0805
- added R7, R8: 2M, microbuilder:0805
- added SDCARD2: ADAFRUIT_SDCARD3V3BOTTOM_MNT, TeelSys-0.3:ADAFRUIT_SDCARD3V3_B
- moved S1 4.23 mm to (42.0, 6.73), flipped to the bottom, turned to 0 degrees
- moved S2 4.23 mm to (42.0, 2.29), flipped to the bottom, turned to 0 degrees
- moved BAT_1 1.23 mm to (61.0, 3.81), flipped to the bottom
- flipped C1 to the bottom
- flipped R1 to the bottom
- flipped R2 to the bottom
- flipped R3 to the bottom, turned to 180 degrees
- flipped R4 to the bottom, turned to 180 degrees
- flipped R5 to the bottom, turned to 180 degrees
- flipped R6 to the bottom, turned to 180 degrees
Connections:
- new net USB_SENSE: C2.2, FEATHER_RP2040.10_D5, R7.2, R8.1
- new net V_USB: FEATHER_RP2040.3_VBUS, R7.1
- net 3.3V: now also SDCARD2.1_3V3; no longer SDCARD1.1_3V3
- net GND: now also C2.1, R8.2, SDCARD2.2_GND; no longer SDCARD1.2_GND
- net N$1: now also SDCARD2.9_CARDDET; no longer SDCARD1.9_CARDDET
- net N$2: now also SDCARD2.4_DO; no longer SDCARD1.4_DO
- net N$3: now also SDCARD2.3_SCLK; no longer SDCARD1.3_SCLK
- net N$4: now also SDCARD2.5_DI; no longer SDCARD1.5_DI
- net N$5: now also SDCARD2.6_CS; no longer SDCARD1.6_CS
Routing:
- net USB_SENSE: track 0.00 -> 29.8 mm, vias 0 -> 2
- net GND: track 155.3 -> 135.1 mm, vias 3 -> 7
- net V_USB: track 0.00 -> 7.30 mm
- net VBAT: track 46.9 -> 42.4 mm, vias 2 -> 1
- net N$17: track 26.0 -> 21.7 mm
- net N$7: track 30.5 -> 28.5 mm
- net N$12: track 67.1 -> 68.0 mm
- net N$4: track 57.5 -> 56.7 mm
- net N$8: track 42.5 -> 42.9 mm, vias 0 -> 2
- net N$10: track 40.0 -> 40.4 mm, vias 0 -> 1
- net N$11: track 40.0 -> 39.7 mm, vias 0 -> 1
- net N$14: track 76.8 -> 77.0 mm, vias 1 -> 3
- net N$9: track 41.0 -> 40.8 mm, vias 0 -> 1
- net N$2: track 40.0 -> 40.1 mm, vias 1 -> 3
- net N$3: vias 1 -> 3
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