File: PCB/main.sch (EAGLE design)
At the start: 19 parts

Commit message: Updated PCB
Parts:
- removed SDCARD1: ADAFRUIT_SDCARD3V3THROUGHHOLE, TeelSys-0.3:ADAFRUIT_SDCARD3V3THROUGHHOLE
- added C2: 0.1 uF, microbuilder:CAP_CERAMIC_0805
- added R7, R8: 2M, microbuilder:RESISTOR0805
- added SDCARD2: ADAFRUIT_SDCARD3V3BOTTOM_MNT, TeelSys-0.3:ADAFRUIT_SDCARD3V3BOTTOM_MNT
Connections:
- new net USB_SENSE: C2.P$2, FEATHER_RP2040.10_D5, R7.2, R8.1
- new net V_USB: FEATHER_RP2040.3_VUSB, R7.1
- net 3.3V: now also SDCARD2.1_3V3; no longer SDCARD1.1_3V3
- net GND: now also C2.P$1, R8.2, SDCARD2.2_GND; no longer SDCARD1.2_GND
- net N$1: now also SDCARD2.9_CARDDET; no longer SDCARD1.9_CARDDET
- net N$2: now also SDCARD2.4_DO; no longer SDCARD1.4_DO
- net N$3: now also SDCARD2.3_SCLK; no longer SDCARD1.3_SCLK
- net N$4: now also SDCARD2.5_DI; no longer SDCARD1.5_DI
- net N$5: now also SDCARD2.6_CS; no longer SDCARD1.6_CS
Changed lines of the file:
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@@
 <part name="FRAME1" library="teelsys-0.2" deviceset="LETTER_L" device=""/>
 <part name="FEATHER_RP2040" library="TeelSys-0.3" deviceset="ADAFRUIT_FEATHER_RP2040" device=""/>
-<part name="SDCARD1" library="TeelSys-0.3" deviceset="ADAFRUIT_SDCARD3V3" device="THROUGHHOLE"/>
 <part name="U$1" library="microbuilder" deviceset="3.3V" device=""/>
 <part name="U$2" library="microbuilder" deviceset="3.3V" device=""/>
@@
 <part name="JSTPH" library="adafruit" deviceset="JST_2PIN" device="-SMT-RA"/>
 <part name="U$13" library="microbuilder" deviceset="GND" device=""/>
+<part name="R7" library="microbuilder" deviceset="RESISTOR" device="0805" value="2M"/>
+<part name="R8" library="microbuilder" deviceset="RESISTOR" device="0805" value="2M"/>
+<part name="C2" library="microbuilder" deviceset="CAP_CERAMIC" device="_0805" value="0.1 uF"/>
+<part name="U$14" library="microbuilder" deviceset="GND" device=""/>
+<part name="SDCARD2" library="TeelSys-0.3" deviceset="ADAFRUIT_SDCARD3V3" device="BOTTOM_MNT"/>
 </parts>
 <sheets>
@@
 <instance part="FRAME1" gate="G$2" x="236.22" y="30.48"/>
 <instance part="FEATHER_RP2040" gate="G$1" x="104.14" y="121.92"/>
-<instance part="SDCARD1" gate="G$1" x="157.48" y="127" rot="R270"/>
 <instance part="U$1" gate="G$1" x="154.94" y="132.08"/>
 <instance part="U$2" gate="G$1" x="76.2" y="157.48"/>
@@
 <instance part="JSTPH" gate="G$1" x="205.74" y="147.32" rot="R180"/>
 <instance part="U$13" gate="G$1" x="215.9" y="134.62"/>
+<instance part="R7" gate="G$1" x="213.36" y="101.6" rot="R90"/>
+<instance part="R8" gate="G$1" x="213.36" y="114.3" rot="R90"/>
+<instance part="C2" gate="G$1" x="223.52" y="114.3"/>
+<instance part="U$14" gate="G$1" x="236.22" y="121.92"/>
+<instance part="SDCARD2" gate="G$1" x="160.02" y="127" rot="R270"/>
 </instances>
 <busses>
@@
 <net name="N$1" class="0">
 <segment>
-<pinref part="SDCARD1" gate="G$1" pin="9_CARDDET"/>
-<wire x1="154.94" y1="83.82" x2="142.24" y2="83.82" width="0.1524" layer="91"/>
+<wire x1="157.48" y1="83.82" x2="142.24" y2="83.82" width="0.1524" layer="91"/>
 <wire x1="142.24" y1="83.82" x2="142.24" y2="99.06" width="0.1524" layer="91"/>
 <pinref part="FEATHER_RP2040" gate="G$1" pin="9_D6"/>
 <wire x1="142.24" y1="99.06" x2="121.92" y2="99.06" width="0.1524" layer="91"/>
+<pinref part="SDCARD2" gate="G$1" pin="9_CARDDET"/>
 </segment>
 </net>
@@
 <wire x1="121.92" y1="119.38" x2="142.24" y2="119.38" width="0.1524" layer="91"/>
 <wire x1="142.24" y1="119.38" x2="142.24" y2="109.22" width="0.1524" layer="91"/>
-<pinref part="SDCARD1" gate="G$1" pin="4_DO"/>
-<wire x1="142.24" y1="109.22" x2="154.94" y2="109.22" width="0.1524" layer="91"/>
+<wire x1="142.24" y1="109.22" x2="157.48" y2="109.22" width="0.1524" layer="91"/>
+<pinref part="SDCARD2" gate="G$1" pin="4_DO"/>
 </segment>
 </net>
@@
 <wire x1="121.92" y1="109.22" x2="139.7" y2="109.22" width="0.1524" layer="91"/>
 <wire x1="139.7" y1="109.22" x2="139.7" y2="114.3" width="0.1524" layer="91"/>
-<pinref part="SDCARD1" gate="G$1" pin="3_SCLK"/>
-<wire x1="139.7" y1="114.3" x2="154.94" y2="114.3" width="0.1524" layer="91"/>
+<wire x1="139.7" y1="114.3" x2="157.48" y2="114.3" width="0.1524" layer="91"/>
+<pinref part="SDCARD2" gate="G$1" pin="3_SCLK"/>
 </segment>
 </net>
@@
 <wire x1="121.92" y1="114.3" x2="134.62" y2="114.3" width="0.1524" layer="91"/>
 <wire x1="134.62" y1="114.3" x2="134.62" y2="104.14" width="0.1524" layer="91"/>
-<pinref part="SDCARD1" gate="G$1" pin="5_DI"/>
-<wire x1="134.62" y1="104.14" x2="154.94" y2="104.14" width="0.1524" layer="91"/>
+<wire x1="134.62" y1="104.14" x2="157.48" y2="104.14" width="0.1524" layer="91"/>
+<pinref part="SDCARD2" gate="G$1" pin="5_DI"/>
 </segment>
 </net>
@@
 <wire x1="129.54" y1="101.6" x2="152.4" y2="101.6" width="0.1524" layer="91"/>
 <wire x1="152.4" y1="101.6" x2="152.4" y2="99.06" width="0.1524" layer="91"/>
-<pinref part="SDCARD1" gate="G$1" pin="6_CS"/>
-<wire x1="152.4" y1="99.06" x2="154.94" y2="99.06" width="0.1524" layer="91"/>
+<pinref part="SDCARD2" gate="G$1" pin="6_CS"/>
+<wire x1="152.4" y1="99.06" x2="157.48" y2="99.06" width="0.1524" layer="91"/>
 </segment>
 </net>
@@
 <wire x1="147.32" y1="129.54" x2="149.86" y2="129.54" width="0.1524" layer="91"/>
 <wire x1="149.86" y1="129.54" x2="149.86" y2="119.38" width="0.1524" layer="91"/>
-<pinref part="SDCARD1" gate="G$1" pin="2_GND"/>
-<wire x1="149.86" y1="119.38" x2="154.94" y2="119.38" width="0.1524" layer="91"/>
+<wire x1="149.86" y1="119.38" x2="157.48" y2="119.38" width="0.1524" layer="91"/>
 <pinref part="S1" gate="1" pin="S"/>
 <wire x1="139.7" y1="132.08" x2="147.32" y2="132.08" width="0.1524" layer="91"/>
 <wire x1="147.32" y1="132.08" x2="147.32" y2="129.54" width="0.1524" layer="91"/>
 <junction x="147.32" y="129.54"/>
+<pinref part="SDCARD2" gate="G$1" pin="2_GND"/>
 </segment>
 <segment>
@@
 <wire x1="215.9" y1="144.78" x2="215.9" y2="137.16" width="0.1524" layer="91"/>
 </segment>
+<segment>
+<pinref part="R8" gate="G$1" pin="2"/>
+<pinref part="C2" gate="G$1" pin="P$1"/>
+<wire x1="213.36" y1="119.38" x2="218.44" y2="119.38" width="0.1524" layer="91"/>
+<pinref part="U$14" gate="G$1" pin="GND"/>
+<wire x1="218.44" y1="119.38" x2="223.52" y2="119.38" width="0.1524" layer="91"/>
+<wire x1="236.22" y1="124.46" x2="218.44" y2="124.46" width="0.1524" layer="91"/>
+<wire x1="218.44" y1="124.46" x2="218.44" y2="119.38" width="0.1524" layer="91"/>
+<junction x="218.44" y="119.38"/>
+</segment>
 </net>
 <net name="3.3V" class="0">
 <segment>
 <pinref part="U$1" gate="G$1" pin="3.3V"/>
-<pinref part="SDCARD1" gate="G$1" pin="1_3V3"/>
 <wire x1="154.94" y1="129.54" x2="154.94" y2="124.46" width="0.1524" layer="91"/>
+<pinref part="SDCARD2" gate="G$1" pin="1_3V3"/>
+<wire x1="154.94" y1="124.46" x2="157.48" y2="124.46" width="0.1524" layer="91"/>
 </segment>
 <segment>
@@
 </segment>
 </net>
+<net name="USB_SENSE" class="0">
+<segment>
+<pinref part="R8" gate="G$1" pin="1"/>
+<pinref part="R7" gate="G$1" pin="2"/>
+<wire x1="213.36" y1="109.22" x2="213.36" y2="106.68" width="0.1524" layer="91"/>
+<pinref part="C2" gate="G$1" pin="P$2"/>
+<wire x1="223.52" y1="111.76" x2="223.52" y2="106.68" width="0.1524" layer="91"/>
+<wire x1="223.52" y1="106.68" x2="213.36" y2="106.68" width="0.1524" layer="91"/>
+<junction x="213.36" y="106.68"/>
+<wire x1="228.6" y1="106.68" x2="223.52" y2="106.68" width="0.1524" layer="91"/>
+<junction x="223.52" y="106.68"/>
+<label x="228.6" y="106.68" size="1.778" layer="95" xref="yes"/>
+</segment>
+<segment>
+<pinref part="FEATHER_RP2040" gate="G$1" pin="10_D5"/>
+<wire x1="121.92" y1="93.98" x2="124.46" y2="93.98" width="0.1524" layer="91"/>
+<label x="124.46" y="93.98" size="1.778" layer="95" xref="yes"/>
+</segment>
+</net>
+<net name="V_USB" class="0">
+<segment>
+<pinref part="FEATHER_RP2040" gate="G$1" pin="3_VUSB"/>
+<wire x1="121.92" y1="129.54" x2="124.46" y2="129.54" width="0.1524" layer="91"/>
+<label x="124.46" y="129.54" size="1.778" layer="95" xref="yes"/>
+</segment>
+<segment>
+<pinref part="R7" gate="G$1" pin="1"/>
+<wire x1="213.36" y1="96.52" x2="213.36" y2="93.98" width="0.1524" layer="91"/>
+<wire x1="213.36" y1="93.98" x2="210.82" y2="93.98" width="0.1524" layer="91"/>
+<label x="210.82" y="93.98" size="1.778" layer="95" rot="R180" xref="yes"/>
+</segment>
+</net>
